File: RoveSoMoCo/RoveSoMoCo.kicad_pcb (KiCad board)
At the start: 4 copper layers, 36.1 x 36.1 mm, 34 parts, among them Q1 SI4156DY, Q2 SI4156DY, Q3 SI4156DY, Q4 SI4156DY, U1 74LVC2G04, U2 IRS2005S, U3 IRS2005S, U4 74HC00

Commit message: Added header and signature
Parts:
- added G***: LOGO, Project Library:z_sig_Malacki_Ehlers_10mmx3mm, F.Cu at (82.5, 63.0)
- added G***: LOGO, Project Library:z_sig_Malacki_Ehlers_23mmx7mm, B.Cu at (128.0, 67.6)
Other:
- board text added: "RoveSoMoCo, Rev1 Mars Rover Design Team Missouri S&T, 2023 Malacki Ehlers"

Commit message: generated gerbs (again)
Parts:
- removed the G*** at (128.0, 67.6)
